File: sparrow_ble/sparrow_ble.sch (EAGLE design)
At the start: 58 parts, among them IC1 SI1145, IC2 TC1262, J3 SMALL_HEADER_5X2, Q3 32768kHz, Q4 FA-128, T1 FDV304P, U1 47491-001, U2 FT232R, U3 NRF51822, U4 SI7020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

Commit message: Add new version with fixed balun
Parts:
- removed C18: 2.2pF, X7R, resistor:C-EUC0402
- removed C19: 1pF, X7R, resistor:C-EUC0402
- removed C20: 1.5pF, X7R, resistor:C-EUC0402
- removed C21: 2.2nF, X7R, resistor:C-EUC0402
- removed D1: BAT54C, diode:BAT54C
- removed L1: 3.3nH, SparkFun-Passives:INDUCTOR0402
- removed L2, L3: 4.7nH, HF, SparkFun-Passives:INDUCTOR0402
- added C17: 2,2nF, resistor:C-EUC0402
- added F1: 2450BM14E0003, johanson:2450BM15A0002
- IC2: value TC1262 -> TC1262-3.3V
Connections:
- net N$17 renamed VBAT
- removed net N$15: C18.2, C19.2, L1.1
- removed net N$22: C20.2, L1.2, U8.P$1
- removed net N$7: D1.A2, U$2.2
- removed net N$8: C8.1, D1.A1, IC2.OUT
- new net N$10: F1.UNBAL, U8.P$1
- new net VLDO: C8.1, IC2.OUT, U$2.1
- net 3.3V: now also U$2.2; no longer D1.CC
- net ANT1: now also F1.BAL@2; no longer L2.2, L3.1
- net ANT2: now also F1.BAL@1; no longer C18.1, L2.1
- net GND: now also C17.2, F1.GND@1, F1.GND@3; no longer C19.1, C20.1, C21.2
- net VDD_PA: now also C17.1, F1.GND@2; no longer C21.1, L3.2
Other:
- note added: "LDO & BAT"
- note added: "MISC"
- note added: "SENSORS"
- note added: "USB TO SERIAL"
- moved on the sheet: C10, C11, C16, C6, C7, C8, C9, IC1, IC2, LED5, LED6, LED7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

Commit message: hw: Update ADC design with values used on actual hardware
Parts:
- R7: value 33k -> 22K
- R8: value 52K3 -> 100K
Other:
- note added: "1.2V reference, 1/3 prescaling"
- note added: "V_bat= (3*1.2)*(ADC/1023)/(100/122)"
- note removed: "1.6V reference"
- note removed: "V_bat= ADC/247.6"
Changed lines of the file:
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@@
 <?xml version="1.0" encoding="utf-8"?>
 <!DOCTYPE eagle SYSTEM "eagle.dtd">
-<eagle version="6.1">
+<eagle version="7.5.0">
 <drawing>
 <settings>
@@
 <setting verticaltext="up"/>
 </settings>
-<grid distance="0.05" unitdist="inch" unit="inch" style="lines" multiple="1" display="no" altdistance="0.01" altunitdist="inch" altunit="inch"/>
+<grid distance="0.1" unitdist="inch" unit="inch" style="lines" multiple="1" display="no" altdistance="0.01" altunitdist="inch" altunit="inch"/>
 <layers>
 <layer number="1" name="Top" color="4" fill="1" visible="no" active="no"/>
@@
 <part name="R5" library="resistor" deviceset="R-EU_" device="R0402" value="10K"/>
 <part name="P+3" library="SparkFun" deviceset="3.3V" device=""/>
-<part name="R8" library="resistor" deviceset="R-EU_" device="R0402" value="52K3"/>
-<part name="R7" library="resistor" deviceset="R-EU_" device="R0402" value="33k"/>
+<part name="R8" library="resistor" deviceset="R-EU_" device="R0402" value="100K"/>
+<part name="R7" library="resistor" deviceset="R-EU_" device="R0402" value="22K"/>
 <part name="GND19" library="supply1" deviceset="GND" device=""/>
 <part name="R11" library="resistor" deviceset="R-EU_" device="R0402" value="10K"/>
@@
 <text x="-22.86" y="58.42" size="6.4516" layer="97" font="vector" ratio="15">NRF51822</text>
 <text x="-129.54" y="121.92" size="6.4516" layer="97" font="vector" ratio="15">CRYSTALS</text>
-<text x="292.227" y="-40.259" size="1.778" layer="91">1.6V reference</text>
-<text x="292.227" y="-42.799" size="1.778" layer="91">10 bit resolution</text>
-<text x="292.227" y="-45.339" size="1.778" layer="91">V_bat= ADC/247.6</text>
+<text x="299.847" y="-22.479" size="1.778" layer="91">1.2V reference, 1/3 prescaling</text>
+<text x="299.847" y="-25.019" size="1.778" layer="91">10 bit resolution</text>
+<text x="299.847" y="-27.559" size="1.778" layer="91">V_bat= (3*1.2)*(ADC/1023)/(100/122)</text>
 <wire x1="-129.54" y1="11.43" x2="113.03" y2="11.43" width="0.8128" layer="97" style="longdash"/>
 <wire x1="113.03" y1="11.43" x2="113.03" y2="-59.69" width="0.8128" layer="97" style="longdash"/>
 <wire x1="113.03" y1="-59.69" x2="-132.08" y2="-59.69" width="0.8128" layer="97" style="longdash"/>
 <wire x1="-132.08" y1="-59.69" x2="-132.08" y2="10.16" width="0.8128" layer="97" style="longdash"/>
-<wire x1="-36.83" y1="-64.77" x2="113.03" y2="-64.77" width="0.8128" layer="97" style="longdash"/>
+<wire x1="-46.99" y1="-64.77" x2="113.03" y2="-64.77" width="0.8128" layer="97" style="longdash"/>
 <wire x1="113.03" y1="-64.77" x2="113.03" y2="-129.54" width="0.8128" layer="97" style="longdash"/>
 <wire x1="113.03" y1="-129.54" x2="-46.99" y2="-129.54" width="0.8128" layer="97" style="longdash"/>
 <wire x1="-46.99" y1="-129.54" x2="-46.99" y2="-64.77" width="0.8128" layer="97" style="longdash"/>
-<wire x1="-46.99" y1="-64.77" x2="-36.83" y2="-64.77" width="0.8128" layer="97" style="longdash"/>
-<wire x1="135.89" y1="12.7" x2="138.43" y2="12.7" width="0.8128" layer="97" style="longdash"/>
-<wire x1="138.43" y1="12.7" x2="379.73" y2="12.7" width="0.8128" layer="97" style="longdash"/>
-<wire x1="379.73" y1="12.7" x2="379.73" y2="-55.88" width="0.8128" layer="97" style="longdash"/>
-<wire x1="379.73" y1="-55.88" x2="379.73" y2="-59.69" width="0.8128" layer="97" style="longdash"/>
+<wire x1="134.62" y1="12.7" x2="379.73" y2="12.7" width="0.8128" layer="97" style="longdash"/>
+<wire x1="379.73" y1="12.7" x2="379.73" y2="-59.69" width="0.8128" layer="97" style="longdash"/>
 <wire x1="379.73" y1="-59.69" x2="134.62" y2="-59.69" width="0.8128" layer="97" style="longdash"/>
 <wire x1="134.62" y1="-59.69" x2="134.62" y2="12.7" width="0.8128" layer="97" style="longdash"/>
-<wire x1="134.62" y1="12.7" x2="138.43" y2="12.7" width="0.8128" layer="97" style="longdash"/>
 <wire x1="135.89" y1="-63.5" x2="297.18" y2="-63.5" width="0.8128" layer="97" style="longdash"/>
 <wire x1="297.18" y1="-63.5" x2="297.18" y2="-129.54" width="0.8128" layer="97" style="longdash"/>
